Commit message: lab07 branched

File: src/husky-kinetic-devel/husky_description/urdf/husky.urdf.xacro (robot description, xacro)
@@ -89,4 +89,39 @@
     <child link="inertial_link" />
   </joint>
+  <!-- <link name="logical_camera_link">
+    <origin xyz="0 0 0.2" rpy="0 0 0" />
+    </link> -->
+    <link name="logical_camera_link">
+        <!-- <collision>
+          <origin xyz="0 0 0" rpy="0 0 0"/>
+        <geometry>
+          <box size="0.1 0.1 0.1"/>
+        </geometry>
+      </collision> -->
+      <visual>
+          <origin xyz="0 0 0" rpy="0 0 0"/>
+          <!-- <origin xyz="0 0 0" rpy="0 0 -3.14"/> -->
+          <!-- <origin xyz="-0.35 0 0.51" rpy="0 0 -3.14"/> -->
+          <geometry>
+            <box size="0.1 0.1 0.1"/>
+          </geometry>
+          <material name="red"/>
+      </visual>
+      <!-- <inertial>
+        <mass value="1e-5" />
+        <origin xyz="0 0 0" rpy="0 0 0"/>
+        <inertia ixx="1e-6" ixy="0" ixz="0" iyy="1e-6" iyz="0" izz="1e-6" />
+      </inertial> -->
+    </link>
+    <!-- <joint name="logical_camera_joint" type="fixed">
+      <parent link="base_link" />
+      <child link="logical_camera_link" />
+    </joint> -->
+    <joint name="logical_camera_joint" type="fixed">
+      <origin xyz="0 0 0" rpy="0 0 0"/>
+      <!-- <axis xyz="0 1 0" /> -->
+      <parent link="top_plate_link"/>
+      <child link="logical_camera_link"/>
+    </joint>
   <!-- IMU Link is the standard mounting position for the UM6 IMU.-->
   <!-- Can be modified with environment variables in /etc/ros/setup.bash -->
@@ -167,4 +202,22 @@
     </plugin>
   </gazebo>
+  <!-- LOGICAL CAMERA SENSOR -->
+  <gazebo reference="logical_camera_link">
+      <sensor name="logical_camera" type="logical_camera">
+          <logical_camera>
+            <near>0.02</near>
+            <far>2</far>
+            <horizontal_fov>0.9</horizontal_fov>
+            <aspect_ratio>0.5</aspect_ratio>
+          </logical_camera>
+          <visualize>true</visualize>
+          <always_on>true</always_on>
+          <update_rate>10</update_rate>
+      </sensor>
+  </gazebo>
+<gazebo>
+    <plugin name="logical_camera" filename="liblogical_camera_plugin.so">
+    </plugin>
+</gazebo>
   <!-- Optional custom includes. -->
   <xacro:include filename="$(arg urdf_extras)" />
